File: PCB/Attendance Management System.kicad_sch (KiCad schematic)
At the start: 0 parts

Commit message: Schematic is almost ready
Other:
- sheet MCU ports: added BAT_SENSE, NFC_IRQ, NFC_MISO, NFC_MOSI, NFC_NSS, NFC_SCK; removed none
- sheet Power ports: added BAT_SENSE; removed none
- sheet RFID ports: added NFC_IRQ, NFC_MISO, NFC_MOSI, NFC_NSS, NFC_SCK; removed none
Changed lines of the file:
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@@
 	(wire
 		(pts
-			(xy 97.79 86.36) (xy 120.65 86.36)
-		)
-		(stroke
-			(width 0)
-			(type default)
-		)
-	)
-	(wire
-		(pts
-			(xy 97.79 90.17) (xy 120.65 90.17)
+			(xy 99.06 93.98) (xy 120.65 93.98)
+		)
+		(stroke
+			(width 0)
+			(type default)
+		)
+	)
+	(wire
+		(pts
+			(xy 167.64 99.06) (xy 187.96 99.06)
+		)
+		(stroke
+			(width 0)
+			(type default)
+		)
+	)
+	(wire
+		(pts
+			(xy 167.64 91.44) (xy 187.96 91.44)
+		)
+		(stroke
+			(width 0)
+			(type default)
+		)
+	)
+	(wire
+		(pts
+			(xy 99.06 86.36) (xy 120.65 86.36)
+		)
+		(stroke
+			(width 0)
+			(type default)
+		)
+	)
+	(wire
+		(pts
+			(xy 167.64 96.52) (xy 187.96 96.52)
+		)
+		(stroke
+			(width 0)
+			(type default)
+		)
+	)
+	(wire
+		(pts
+			(xy 167.64 104.14) (xy 187.96 104.14)
+		)
+		(stroke
+			(width 0)
+			(type default)
+		)
+	)
+	(wire
+		(pts
+			(xy 167.64 93.98) (xy 187.96 93.98)
+		)
+		(stroke
+			(width 0)
+			(type default)
+		)
+	)
+	(wire
+		(pts
+			(xy 99.06 90.17) (xy 120.65 90.17)
 		)
 		(stroke
@@
 			)
 		)
+		(pin "NFC_MISO" input
+			(at 167.64 96.52 0)
+			(effects
+				(font
+					(size 1.27 1.27)
+				)
+				(justify right)
+			)
+		)
+		(pin "NFC_MOSI" output
+			(at 167.64 93.98 0)
+			(effects
+				(font
+					(size 1.27 1.27)
+				)
+				(justify right)
+			)
+		)
+		(pin "NFC_NSS" output
+			(at 167.64 91.44 0)
+			(effects
+				(font
+					(size 1.27 1.27)
+				)
+				(justify right)
+			)
+		)
+		(pin "NFC_IRQ" input
+			(at 167.64 104.14 0)
+			(effects
+				(font
+					(size 1.27 1.27)
+				)
+				(justify right)
+			)
+		)
+		(pin "NFC_SCK" output
+			(at 167.64 99.06 0)
+			(effects
+				(font
+					(size 1.27 1.27)
+				)
+				(justify right)
+			)
+		)
+		(pin "BAT_SENSE" bidirectional
+			(at 120.65 93.98 180)
+			(effects
+				(font
+					(size 1.27 1.27)
+				)
+				(justify left)
+			)
+		)
 		(instances
 			(project "Attendance Management System"
@@
 	)
 	(sheet
-		(at 76.835 81.915)
-		(size 20.955 13.335)
+		(at 76.835 83.82)
+		(size 22.225 11.43)
 		(exclude_from_sim no)
 		(in_bom yes)
@@
 		)
 		(property "Sheetname" "Power"
-			(at 76.835 81.2034 0)
+			(at 76.835 83.1084 0)
 			(show_name no)
 			(do_not_autoplace no)
@@
 		)
 		(pin "D-" bidirectional
-			(at 97.79 90.17 0)
+			(at 99.06 90.17 0)
 			(effects
 				(font
@@
 		)
 		(pin "D+" bidirectional
-			(at 97.79 86.36 0)
+			(at 99.06 86.36 0)
+			(effects
+				(font
+					(size 1.27 1.27)
+				)
+				(justify right)
+			)
+		)
+		(pin "BAT_SENSE" bidirectional
+			(at 99.06 93.98 0)
 			(effects
 				(font
@@
 	)
 	(sheet
-		(at 205.74 88.9)
-		(size 25.4 20.32)
+		(at 187.96 87.63)
+		(size 25.4 19.05)
 		(exclude_from_sim no)
 		(in_bom yes)
@@
 		)
 		(property "Sheetname" "RFID"
-			(at 205.74 88.1884 0)
+			(at 187.96 86.9184 0)
 			(show_name no)
 			(do_not_autoplace no)
@@
 		)
 		(property "Sheetfile" "rfid.kicad_sch"
-			(at 205.74 109.8046 0)
+			(at 187.96 107.2646 0)
 			(show_name no)
 			(do_not_autoplace no)
@@
 			)
 		)
+		(pin "NFC_NSS" input
+			(at 187.96 91.44 180)
+			(effects
+				(font
+					(size 1.27 1.27)
+				)
+				(justify left)
+			)
+		)
+		(pin "NFC_MOSI" input
+			(at 187.96 93.98 180)
+			(effects
+				(font
+					(size 1.27 1.27)
+				)
+				(justify left)
+			)
+		)
+		(pin "NFC_IRQ" output
+			(at 187.96 104.14 180)
+			(effects
+				(font
+					(size 1.27 1.27)
+				)
+				(justify left)
+			)
+		)
+		(pin "NFC_MISO" output
+			(at 187.96 96.52 180)
+			(effects
+				(font
+					(size 1.27 1.27)
+				)
+				(justify left)
+			)
+		)
+		(pin "NFC_SCK" input
+			(at 187.96 99.06 180)
+			(effects
+				(font
+					(size 1.27 1.27)
+				)
+				(justify left)
+			)
+		)
