File: PCB/Attendance Management System.kicad_sch (KiCad schematic)
At the start: 0 parts

Commit message: ESD diodes added
Other:
- title: (none) -> Card Attendance System
Changed lines of the file:
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@@
 	(generator_version "10.0")
 	(paper "A4")
+	(title_block
+		(title "Card Attendance System")
+		(date "2026-09-25")
+		(rev "0.1")
+		(comment 1 "Top level: power, MCU and NFC reader sheets")
+	)
 	(text "Top"
 		(exclude_from_sim no)
