File: PCB/mcu.kicad_sch (KiCad schematic)
At the start: 24 parts, among them J3 SW, J4 MOT, Q1 AO3400A, SW1 RST, SW2 BOOT, SW3 KEY, U1 STM32L432KCUx, Y2 32kHz

Commit message: Schematic is almost ready
Parts:
- added D4: SS14, Diode_SMD:D_SMA, symbol Diode:SS14
- added R18, R19: 4M7, Resistor_SMD:R_0805_2012Metric, symbol Device:R
- FB1: value FerriteBead -> FB 600 Ohm @ 100MHz
Connections:
- net BAT+: now also D4.1 (K)
- net GND: now also R19.2
- net KEY: now also U1.6 (PA0)
- net at J4.2 (Pin_2), Q1.3 (D): now also D4.2 (A)
- net BAT_SENSE: now reaches U1.13 (PA7)
- net BAT_SENSE: now also U1.30 (PB7)
- net NFC_NSS: now reaches U1.14 (PB0)
- net NFC_IRQ: now reaches U1.15 (PB1)
- net VBUS: now reaches U1.19 (PA9)
- net VBUS: now also R18.2, R19.1
- net NFC_SCK: now reaches U1.26 (PB3)
- net NFC_MISO: now reaches U1.27 (PB4)
- net NFC_MOSI: now reaches U1.28 (PB5)
- net OSC_IN renamed LSC_IN
- net OSC_OUT renamed LSC_OUT
- new net +5V: R18.1
Other:
- moved on the sheet: C1, C2, C3, C4, C5, C6, C7, C8, D5, D6, FB1, J3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
