File: PCB/mcu.kicad_sch (KiCad schematic)
At the start: 27 parts, among them J3 SW, J4 MOT, Q1 AO3400A, SW1 RST, SW2 BOOT, SW3 KEY, U1 STM32L432KCUx, Y2 32kHz

Commit message: PN532 pins are added
Parts:
- added J7: PN532, Connector_PinSocket_2.54mm:PinSocket_1x08_P2.54mm_Vertical, symbol Connector:Conn_01x08_Socket
- added R20: 10K, Resistor_SMD:R_0805_2012Metric, symbol Device:R
Connections:
- net +3V3: now also R20.1
- net BAT+: now also J7.5 (Pin_5)
- net GND: now also J7.6 (Pin_6)
- net NFC_MISO: now also J7.2 (Pin_2)
- net NFC_MOSI: now also J7.3 (Pin_3)
- net NFC_SCK: now also J7.1 (Pin_1)
- net PN532_NSS: now reaches U1.25 (PA15)
- net PN532_NSS: now also J7.4 (Pin_4), R20.2
- net PN532_IRQ: now reaches U1.29 (PB6)
- net PN532_IRQ: now also J7.7 (Pin_7)
- no-connect marks 0 -> 1
Other:
- note added: "PN532 backup reader on SPI1 (Elechouse V3 pinout, DIP = SPI). Own CS on PA15 and IRQ on PB6; SPI mode 0, LSB first, <= 5 MHz."

Commit message: ESD diodes added
Parts:
- C1, C3, C4, C8: Dielectric (none) -> X7R; Voltage (none) -> 16V
- C2, C5: Dielectric (none) -> X5R; Voltage (none) -> 10V
- C6, C7: Dielectric (none) -> C0G; Voltage (none) -> 50V
- FB1: value FB 600 Ohm @ 100MHz -> 600R@100MHz
- J3: value SW -> SWD
- J4: value MOT -> VIB_MOTOR
- R10, R9: value 470 -> 470R
- R11, R20, R7, R8: value 10K -> 10k
- R18, R19: value 4M7 -> 4.7M
- SW2: value BOOT -> BOOT0
- SW3: value KEY -> POWER
- Y2: value 32kHz -> 32.768k
Connections:
- no-connect marks 1 -> 6
Other:
- note added: "32.768 kHz LSE CRYSTAL"
- note added: "MCU DECOUPLING"
- note added: "MICROCONTROLLER STM32L432KC"
- note added: "PN532 BACKUP READER HEADER"
- note added: "PN532 backup reader (Elechouse V3, DIP = SPI). Own CS on PA15, IRQ on PB6 (active low). SPI mode 0, LSB first, max 5 MHz."
- note added: "RESET, BOOT0 AND POWER BUTTONS"
- note added: "STATUS LEDS"
- note added: "SWD DEBUG HEADER"
- note added: "USB VBUS SENSE"
- note added: "VIBRATION MOTOR DRIVER"
- note removed: "PN532 backup reader on SPI1 (Elechouse V3 pinout, DIP = SPI). Own CS on PA15 and IRQ on PB6; SPI mode 0, LSB first, <= 5 MHz."
- title: (none) -> Card Attendance System

Commit message: almost ready for fabrication
Parts:
- C10: renamed from C7; value 4.3p -> 8.2p; LCSC (none) -> C1840
- C11: renamed from C6; value 4.3p -> 8.2p; LCSC (none) -> C1840
- C4: renamed from C2; LCSC (none) -> C1779
- C5: renamed from C8; LCSC (none) -> C49678
- C6: renamed from C1; LCSC (none) -> C49678
- C7: renamed from C3; LCSC (none) -> C49678
- C8: renamed from C4; LCSC (none) -> C1710
- C9: renamed from C5; LCSC (none) -> C28323
- D4: LCSC (none) -> C2480
- D5: LCSC (none) -> C84256
- D6: LCSC (none) -> C98221
- FB1: LCSC (none) -> C76884
- J3: renamed from J7; LCSC (none) -> C42431840
- J4: LCSC (none) -> C492401
- J5: renamed from J3; LCSC (none) -> C2691448
- Q1: LCSC (none) -> C20917
- R10: renamed from R19; LCSC (none) -> C17674
- R11: renamed from R20; LCSC (none) -> C17414
- R12: renamed from R7; LCSC (none) -> C17414
- R13: renamed from R8; LCSC (none) -> C17414
- R14: renamed from R9; LCSC (none) -> C17710
- R15: renamed from R10; LCSC (none) -> C17710
- R16: renamed from R11; LCSC (none) -> C17414
- R9: renamed from R18; LCSC (none) -> C17674
- SW1, SW2, SW3: LCSC (none) -> C2689642
- U4: renamed from U1; value STM32L432KCUx -> STM32L432KBUx; symbol MCU_ST_STM32L4:STM32L432KCUx -> MCU_ST_STM32L4:STM32L432KBUx; LCSC (none) -> C2928224
- Y1: renamed from Y2; LCSC (none) -> C95361
Other:
- note added: "MICROCONTROLLER STM32L432KB"
- note removed: "MICROCONTROLLER STM32L432KC"
