File: PCB/power.kicad_sch (KiCad schematic)
At the start: 14 parts, among them J1 USB_C_Receptacle_USB2.0_16P, J2 BAT, U2 MCP73833-xxx-UN, U3 TPS7A0233PDBVR

Commit message: Schematic is almost ready
Parts:
- added C34: 100n, Capacitor_SMD:C_0805_2012Metric, symbol Device:C
- added R16: 4M7, Resistor_SMD:R_0805_2012Metric, symbol Device:R
- added R17: 2M7, Resistor_SMD:R_0805_2012Metric, symbol Device:R
Connections:
- net BAT+: now also R16.1
- net GND: now also C34.2, R17.2
- new net BAT_SENSE: C34.1, R16.2, R17.1
