File: PCB/power.kicad_sch (KiCad schematic)
At the start: 17 parts, among them J1 USB_C_Receptacle_USB2.0_16P, J2 BAT, U2 MCP73833-xxx-UN, U3 TPS7A0233PDBVR

Commit message: Schematic is almost ready
Parts:
- added C35: 4.7u, Capacitor_SMD:C_0805_2012Metric, symbol Device:C
- added C36: 10u, Capacitor_SMD:C_0805_2012Metric, symbol Device:C
Connections:
- net +5V: now also C35.1
- net BAT+: now also C36.1
- net GND: now also C35.2, C36.2

Commit message: ESD diodes added
Parts:
- added U6: USBLC6-2SC6, Package_TO_SOT_SMD:SOT-23-6, symbol Power_Protection:USBLC6-2SC6
- C34: Dielectric (none) -> X7R; Voltage (none) -> 16V
- C35: Dielectric (none) -> X5R; Voltage (none) -> 16V
- C36: Dielectric (none) -> X5R; Voltage (none) -> 10V
- J1: value USB_C_Receptacle_USB2.0_16P -> USB-C
- J2: value BAT -> BATTERY
- R1, R2: value 5K1 -> 5.1k
- R16: value 4M7 -> 4.7M
- R17: value 2M7 -> 2.7M
- R3, R4, R5: value 470 -> 470R
- R6: value 1K -> 1k
- TH1: value Therm_NTC -> 10k NTC
Connections:
- net +5V: now also U6.5 (VBUS)
- net D+: now also U6.1 (I/O1), U6.6 (I/O1)
- net D-: now also U6.3 (I/O2), U6.4 (I/O2)
- net GND: now also U6.2 (GND)
Other:
- note added: "3.3 V LDO TPS7A02"
- note added: "BATTERY CONNECTOR"
- note added: "BATTERY SENSE DIVIDER"
- note added: "BULK CAPACITORS"
- note added: "LI-ION CHARGER MCP73833"
- note added: "Place U6 next to J1 and route D+/D- straight through its pads."
- note added: "USB ESD PROTECTION"
- note added: "USB-C INPUT (SINK)"
- title: (none) -> Card Attendance System

Commit message: almost ready for fabrication
Parts:
- C1: renamed from C35; LCSC (none) -> C1779
- C2: renamed from C36; LCSC (none) -> C15850
- C3: renamed from C34; LCSC (none) -> C49678
- D1: renamed from D3; LCSC (none) -> C98221
- D2: LCSC (none) -> C98221
- D3: renamed from D1; LCSC (none) -> C84256
- J1: LCSC (none) -> C5143397
- J2: LCSC (none) -> C263753
- R1, R2: LCSC (none) -> C27834
- R3, R4, R5: LCSC (none) -> C17710
- R6: LCSC (none) -> C17513
- R7: renamed from R16; LCSC (none) -> C17674
- R8: renamed from R17; LCSC (none) -> C17531
- TH1: LCSC (none) -> C141588
- U1: renamed from U6; LCSC (none) -> C7519
- U2: LCSC (none) -> C627668
- U3: LCSC (none) -> C2887324
