File: PCB/rfid.kicad_sch (KiCad schematic)
At the start: 38 parts, among them U4 ST25R3916-AQWT, Y1 27.120 MHz

Commit message: Schematic is almost ready
Parts:
- removed L1, L2: 470 nH, Package_SO:SOIC-20W_7.5x12.8mm_P1.27mm, symbol Device:L
- removed Pad_CSI1, Pad_CSO1: Conn_01x01_Pin, symbol Connector:Conn_01x01_Pin
- added J5: CS01, Connector_Wire:SolderWirePad_1x01_SMD_1x2mm, symbol Connector:Conn_01x01_Pin
- added J6: CSI1, Connector_Wire:SolderWirePad_1x01_SMD_1x2mm, symbol Connector:Conn_01x01_Pin
- added L3, L4: 470n, Inductor_SMD:L_0402_1005Metric, symbol Device:L
- AE1: footprint Package_DFN_QFN:DFN-8-1EP_2x3mm_P0.5mm_EP0.61x2.2mm -> (none)
- C10, C11, C12, C13, C14, C15, C16, C17, C18, C19, C20, C21, C22, C23, C24, C25, C26, C27, C28, C29, C30, C31, C32, C33, C9: footprint (none) -> Capacitor_SMD:C_0805_2012Metric
- FB2: value 600 Ohm @ 100MHz -> FB 600 Ohm @ 100MHz; footprint Package_LCC:PLCC-84_29.3x29.3mm_P1.27mm -> Inductor_SMD:L_0402_1005Metric
- R12, R13, R14, R15: footprint Package_QFP:LQFP-32_7x7mm_P0.8mm -> Resistor_SMD:R_0805_2012Metric
- U4: footprint ST25R3916-AQWT:QFN50P500X500X100-33N -> External:QFN50P500X500X100-33N
- Y1: value 27.120 MHz -> ABM8-27.120MHZ; footprint Oscillator:Oscillator_DIP-14 -> Crystal:Crystal_SMD_3225-4Pin_3.2x2.5mm_HandSoldering
Connections:
- net +3V3: now also FB2.2; no longer FB2.1
- net AN1: now also L3.1
- net AN2: now also L4.1
- net DC1: now also FB2.1; no longer FB2.2
- net at C12.1, C16.2: now also L3.2
- net at U4.2 (CSO): now also J5.1 (Pin_1)
- net at U4.25 (CSI): now also J6.1 (Pin_1)
- net at C13.1, C17.2: now also L4.2
