File: PCB/Attendance Management System.kicad_pcb (KiCad board)
At the start: 2 copper layers, 10 parts, among them J1 USB_C_Receptacle_USB2.0_16P, U1 STM32L432KCUx, U2 MCP73833-xxx-UN

Commit message: Schematic is almost ready
Parts:
- added AE1: Antenna, Package_DFN_QFN:DFN-8-1EP_2x3mm_P0.5mm_EP0.61x2.2mm, F.Cu at (151.4, 77.3)
- added C10: 15pF, Capacitor_SMD:C_0805_2012Metric, F.Cu at (151.5, 58.5)
- added C11: 100nF, Capacitor_SMD:C_0805_2012Metric, F.Cu at (151.5, 61.5)
- added C12: 150 pF, Capacitor_SMD:C_0805_2012Metric, F.Cu at (151.5, 64.5)
- added C13: 150 pF, Capacitor_SMD:C_0805_2012Metric, F.Cu at (151.5, 67.5)
- added C14: 100 pF, Capacitor_SMD:C_0805_2012Metric, F.Cu at (151.5, 70.5)
- added C15: 100 pF, Capacitor_SMD:C_0805_2012Metric, F.Cu at (151.5, 73.5)
- added C16: 68 pF, Capacitor_SMD:C_0805_2012Metric, F.Cu at (155.9, 55.5)
- added C17: 68 pF, Capacitor_SMD:C_0805_2012Metric, F.Cu at (155.9, 58.5)
- added C18: 270 pF, Capacitor_SMD:C_0805_2012Metric, F.Cu at (155.9, 61.5)
- added C19: 270 pF, Capacitor_SMD:C_0805_2012Metric, F.Cu at (155.9, 64.5)
- added C20: 10uF, Capacitor_SMD:C_0805_2012Metric, F.Cu at (155.9, 67.5)
- added C21: 10uF, Capacitor_SMD:C_0805_2012Metric, F.Cu at (155.9, 70.5)
- added C22: 100 nF, Capacitor_SMD:C_0805_2012Metric, F.Cu at (155.9, 73.5)
- added C23: 100 nF, Capacitor_SMD:C_0805_2012Metric, F.Cu at (160.4, 55.5)
- added C24: 100nF, Capacitor_SMD:C_0805_2012Metric, F.Cu at (160.4, 58.5)
- added C25: 100nF, Capacitor_SMD:C_0805_2012Metric, F.Cu at (160.4, 61.5)
- added C26: 2.2uF, Capacitor_SMD:C_0805_2012Metric, F.Cu at (160.4, 64.5)
- added C27: 2.2uF, Capacitor_SMD:C_0805_2012Metric, F.Cu at (160.4, 67.5)
- added C28: 100 nF, Capacitor_SMD:C_0805_2012Metric, F.Cu at (160.4, 70.5)
- added C29: 100 nF, Capacitor_SMD:C_0805_2012Metric, F.Cu at (160.4, 73.5)
- added C30: 100 nF, Capacitor_SMD:C_0805_2012Metric, F.Cu at (164.8, 55.5)
- added C31: 2.2uF, Capacitor_SMD:C_0805_2012Metric, F.Cu at (164.8, 58.5)
- added C32: 2.2uF, Capacitor_SMD:C_0805_2012Metric, F.Cu at (164.8, 61.5)
- added C33: 1 uF, Capacitor_SMD:C_0805_2012Metric, F.Cu at (164.8, 64.5)
- added C34: 100n, Capacitor_SMD:C_0805_2012Metric, F.Cu at (185.2, 70.0)
- added C6: 4.3p, Capacitor_SMD:C_0805_2012Metric, F.Cu at (181.8, 38.6)
- added C7: 4.3p, Capacitor_SMD:C_0805_2012Metric, F.Cu at (181.8, 41.6)
- added C8: 100n, Capacitor_SMD:C_0805_2012Metric, F.Cu at (181.8, 44.6)
- added C9: 15pF, Capacitor_SMD:C_0805_2012Metric, F.Cu at (151.5, 55.5)
- added D1: RED, LED_SMD:LED_0805_2012Metric, F.Cu at (190.1, 52.2)
- added D2: GREEN, LED_SMD:LED_0805_2012Metric, F.Cu at (190.1, 55.3)
- added D3: GREEN, LED_SMD:LED_0805_2012Metric, F.Cu at (190.1, 58.3)
- added D4: SS14, Diode_SMD:D_SMA, F.Cu at (201.6, 29.8)
- added D5: RED, LED_SMD:LED_0805_2012Metric, F.Cu at (186.3, 44.2)
- added D6: GREEN, LED_SMD:LED_0805_2012Metric, F.Cu at (186.3, 47.2)
- added FB1: FB 600 Ohm @ 100MHz, Inductor_SMD:L_0402_1005Metric, F.Cu at (175.7, 46.1)
- added FB2: FB 600 Ohm @ 100MHz, Inductor_SMD:L_0402_1005Metric, F.Cu at (141.5, 13.0)
- added J2: BAT, Connector_JST:JST_XA_B02B-XASK-1_1x02_P2.50mm_Vertical, F.Cu at (177.0, 64.9)
- added J3: SW, Connector_PinHeader_2.54mm:PinHeader_1x04_P2.54mm_Vertical, F.Cu at (190.7, 24.3)
- added J4: MOT, Connector_PinHeader_2.54mm:PinHeader_1x02_P2.54mm_Vertical, F.Cu at (190.7, 36.5)
- added J5: CS01, Connector_Wire:SolderWirePad_1x01_SMD_1x2mm, F.Cu at (134.0, 40.3)
- added J6: CSI1, Connector_Wire:SolderWirePad_1x01_SMD_1x2mm, F.Cu at (136.6, 40.3)
- added L3: 470n, Inductor_SMD:L_0402_1005Metric, F.Cu at (128.0, 56.0)
- added L4: 470n, Inductor_SMD:L_0402_1005Metric, F.Cu at (128.0, 58.0)
- added Q1: AO3400A, Package_TO_SOT_SMD:SOT-23, F.Cu at (190.9, 44.9)
- added R10: 470, Resistor_SMD:R_0805_2012Metric, F.Cu at (186.2, 32.3)
- added R11: 10K, Resistor_SMD:R_0805_2012Metric, F.Cu at (186.2, 35.3)
- added R12: 10k, Resistor_SMD:R_0805_2012Metric, F.Cu at (117.7, 27.7)
- added R13: 1 KOhm, Resistor_SMD:R_0805_2012Metric, F.Cu at (117.7, 39.1)
- added R14: 1 KOhm, Resistor_SMD:R_0805_2012Metric, F.Cu at (117.7, 50.5)
- added R15: 1.5 KOhm, Resistor_SMD:R_0805_2012Metric, F.Cu at (117.7, 61.9)
- added R16: 4M7, Resistor_SMD:R_0805_2012Metric, F.Cu at (171.2, 69.9)
- added R17: 2M7, Resistor_SMD:R_0805_2012Metric, F.Cu at (171.2, 72.9)
- added R18: 4M7, Resistor_SMD:R_0805_2012Metric, F.Cu at (186.2, 38.2)
- added R19: 4M7, Resistor_SMD:R_0805_2012Metric, F.Cu at (186.2, 41.2)
- added R3: 470, Resistor_SMD:R_0805_2012Metric, F.Cu at (171.2, 58.1)
- added R4: 470, Resistor_SMD:R_0805_2012Metric, F.Cu at (171.2, 61.1)
- added R5: 470, Resistor_SMD:R_0805_2012Metric, F.Cu at (171.2, 64.0)
- added R6: 1K, Resistor_SMD:R_0805_2012Metric, F.Cu at (171.2, 67.0)
- added R7: 10K, Resistor_SMD:R_0805_2012Metric, F.Cu at (186.2, 23.5)
- added R8: 10K, Resistor_SMD:R_0805_2012Metric, F.Cu at (186.2, 26.4)
- added R9: 470, Resistor_SMD:R_0805_2012Metric, F.Cu at (186.2, 29.4)
- added SW1: RST, Button_Switch_SMD:SW_Tactile_SPST_NO_Straight_CK_PTS636Sx25SMTRLFS, F.Cu at (174.3, 24.6)
- added SW2: BOOT, Button_Switch_SMD:SW_Tactile_SPST_NO_Straight_CK_PTS636Sx25SMTRLFS, F.Cu at (174.3, 29.9)
- added SW3: KEY, Button_Switch_SMD:SW_Tactile_SPST_NO_Straight_CK_PTS636Sx25SMTRLFS, F.Cu at (174.3, 35.1)
- added TH1: Therm_NTC, Resistor_THT:R_Axial_DIN0204_L3.6mm_D1.6mm_P1.90mm_Vertical, F.Cu at (184.6, 66.9)
- added U3: TPS7A0233PDBVR, External:SOT23_DBV_TEX-L, F.Cu at (175.9, 71.5)
- added U4: ST25R3916-AQWT, External:QFN50P500X500X100-33N, F.Cu at (163.7, 38.1)
- added Y1: ABM8-27.120MHZ, Crystal:Crystal_SMD_3225-4Pin_3.2x2.5mm_HandSoldering, F.Cu at (154.6, 38.9)
- added Y2: 32kHz, Crystal:Crystal_SMD_EuroQuartz_EQ161-2Pin_3.2x1.5mm, F.Cu at (171.7, 46.8)
- moved C1 68.4 mm to (181.8, 23.5)
- moved C2 68.4 mm to (181.8, 26.5)
- moved C3 68.4 mm to (181.8, 29.5)
- moved C4 68.4 mm to (181.8, 32.5)
- moved C5 68.4 mm to (181.8, 35.5)
- moved J1 49.5 mm to (180.7, 56.0)
- moved U1 48.2 mm to (173.1, 41.4)
- moved R1 44.5 mm to (171.2, 52.2)
- moved R2 44.5 mm to (171.2, 55.2)
- moved U2 30.0 mm to (186.6, 63.0)
Connections:
- net Net-(U2-V_{BAT}-Pad10) renamed BAT+
- J1 pad A6: /D+ -> /MCU/D+
- J1 pad A7: /D- -> /MCU/D-
- J1 pad B6: /D+ -> /MCU/D+
- J1 pad B7: /D- -> /MCU/D-
- U1 pad 10: unconnected-(U1-PA4-Pad10) -> /MCU/VIB_EN
- U1 pad 13: unconnected-(U1-PA7-Pad13) -> /MCU/BAT_SENSE
- U1 pad 14: unconnected-(U1-PB0-Pad14) -> /MCU/NFC_NSS
- U1 pad 15: unconnected-(U1-PB1-Pad15) -> /MCU/NFC_IRQ
- U1 pad 19: unconnected-(U1-PA9-Pad19) -> /MCU/VBUS
- U1 pad 2: unconnected-(U1-PC14-Pad2) -> /MCU/LSC_IN
- U1 pad 21: unconnected-(U1-PA11-Pad21) -> /MCU/D-
- U1 pad 22: unconnected-(U1-PA12-Pad22) -> /MCU/D+
- U1 pad 23: unconnected-(U1-PA13-Pad23) -> /MCU/SWDIO
- U1 pad 24: unconnected-(U1-PA14-Pad24) -> /MCU/SWCLK
- U1 pad 26: unconnected-(U1-PB3-Pad26) -> /MCU/NFC_SCK
- U1 pad 27: unconnected-(U1-PB4-Pad27) -> /MCU/NFC_MISO
- U1 pad 28: unconnected-(U1-PB5-Pad28) -> /MCU/NFC_MOSI
- U1 pad 3: unconnected-(U1-PC15-Pad3) -> /MCU/LSC_OUT
- U1 pad 30: unconnected-(U1-PB7-Pad30) -> /MCU/BAT_SENSE
- U1 pad 31: unconnected-(U1-PH3-Pad31) -> /MCU/BOOT
- U1 pad 4: unconnected-(U1-NRST-Pad4) -> /MCU/nRST
- U1 pad 6: unconnected-(U1-PA0-Pad6) -> /MCU/KEY
- U1 pad 8: unconnected-(U1-PA2-Pad8) -> /MCU/LED_G
- U1 pad 9: unconnected-(U1-PA3-Pad9) -> /MCU/LED_R
- U2 pad 1: Net-(U2-V_{DD}-Pad1) -> +5V
- U2 pad 2: Net-(U2-V_{DD}-Pad1) -> +5V
- U2 pad 3: unconnected-(U2-STAT1-Pad3) -> Net-(U2-STAT1)
- U2 pad 4: unconnected-(U2-STAT2-Pad4) -> Net-(U2-STAT2)
- U2 pad 5: unconnected-(U2-V_{SS}-Pad5) -> GND
- U2 pad 6: unconnected-(U2-PROG-Pad6) -> Net-(U2-PROG)
- U2 pad 7: unconnected-(U2-~{PG}-Pad7) -> Net-(U2-~{PG})
- U2 pad 8: unconnected-(U2-THERM-Pad8) -> Net-(U2-THERM)

Commit message: Components placed roughly
Parts:
- removed AE1: Antenna, Package_DFN_QFN:DFN-8-1EP_2x3mm_P0.5mm_EP0.61x2.2mm
- removed U4: ST25R3916-AQWT, External:QFN50P500X500X100-33N
- added C35: 4.7u, Capacitor_SMD:C_0805_2012Metric, F.Cu at (126.2, 132.0)
- added C36: 10u, Capacitor_SMD:C_0805_2012Metric, F.Cu at (151.0, 133.9)
- added J7: PN532, Connector_PinSocket_2.54mm:PinSocket_1x08_P2.54mm_Vertical, F.Cu at (103.5, 139.4)
- added R20: 10k, Resistor_SMD:R_0805_2012Metric, F.Cu at (135.1, 115.7)
- added U5: ST25R3916-AQWT, External:QFN50P500X500X100-33N, F.Cu at (130.8, 98.0)
- added U6: USBLC6-2SC6, Package_TO_SOT_SMD:SOT-23-6, F.Cu at (130.0, 133.1)
- C10, C9: value 15pF -> 15p
- C11, C24, C25: value 100nF -> 100n
- C12, C13: value 150 pF -> 150p
- C14, C15: value 100 pF -> 100p
- C16, C17: value 68 pF -> 68p
- C18, C19: value 270 pF -> 270p
- C20, C21: value 10uF -> 10u
- C22, C23, C28, C29, C30: value 100 nF -> 100n
- C26, C27, C31, C32: value 2.2uF -> 2.2u
- C33: value 1 uF -> 1u
- FB1, FB2: value FB 600 Ohm @ 100MHz -> 600R@100MHz
- J1: value USB_C_Receptacle_USB2.0_16P -> USB-C
- J2: value BAT -> BATTERY
- J3: value SW -> SWD
- J4: value MOT -> VIB_MOTOR
- J5: value CS01 -> CSO
- J6: value CSI1 -> CSI
- L3, L4: value 470n -> 470nH
- R1, R2: value 5K1 -> 5.1k
- R10, R3, R4, R5, R9: value 470 -> 470R
- R11, R7, R8: value 10K -> 10k
- R13, R14: value 1 KOhm -> 1k
- R15: value 1.5 KOhm -> 1.5k
- R16, R18, R19: value 4M7 -> 4.7M
- R17: value 2M7 -> 2.7M
- R6: value 1K -> 1k
- SW2: value BOOT -> BOOT0
- SW3: value KEY -> POWER
- TH1: value Therm_NTC -> 10k NTC
- Y1: value ABM8-27.120MHZ -> 27.12MHz
- Y2: value 32kHz -> 32.768k
- moved SW1 119.3 mm to (105.3, 122.0), turned to 90 degrees
- moved R7 112.7 mm to (108.7, 105.3), turned to 90 degrees
- moved R8 111.6 mm to (105.3, 103.2), turned to -90 degrees
- moved C1 109.6 mm to (124.6, 117.0), turned to 180 degrees
- moved C2 107.0 mm to (143.2, 126.3), turned to 180 degrees
- moved C4 104.2 mm to (124.6, 119.7), turned to 180 degrees
- moved C5 103.6 mm to (125.6, 122.6), turned to -90 degrees
- moved D1 103.4 mm to (140.6, 143.0)
- moved C8 101.9 mm to (109.1, 116.0), turned to 90 degrees
- moved SW3 101.8 mm to (105.3, 110.0), turned to 90 degrees
- moved C3 100.5 mm to (135.4, 118.6)
- moved C6 99.8 mm to (121.1, 117.8), turned to -90 degrees
- moved D4 99.6 mm to (152.6, 116.5), turned to -90 degrees
- moved D2 99.1 mm to (144.1, 143.0)
- moved J1 98.8 mm to (130.0, 140.8)
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Connections:
- C21 pad 1: +3V3 -> BAT+
- C25 pad 1: +3V3 -> BAT+
- FB2 pad 2: +3V3 -> BAT+
- U1 pad 25: unconnected-(U1-PA15-Pad25) -> /MCU/PN532_NSS
- U1 pad 29: unconnected-(U1-PB6-Pad29) -> /MCU/PN532_IRQ
Other:
- board outline added: 60 x 105 mm
- board text added: "NFC ANTENNA AREA (loop coil here, no copper pour) feed: DR2 left / DR1 right at the bottom-centre"

Commit message: Routing zones completed|
Parts:
- moved J3 59.3 mm to (104.5, 127.3), turned to 180 degrees
- moved R10 46.2 mm to (120.5, 125.0)
- moved D6 45.9 mm to (120.5, 128.5)
- moved J7 43.4 mm to (130.6, 105.5), turned to -90 degrees
- moved D5 42.3 mm to (123.0, 128.5)
- moved R9 40.8 mm to (123.0, 125.0)
- moved R7 37.4 mm to (116.0, 142.0), turned to -90 degrees
- moved SW2 32.9 mm to (112.0, 139.0), turned to 90 degrees
- moved C19 32.7 mm to (150.4, 99.5), turned to 90 degrees
- moved R15 32.6 mm to (152.4, 104.5), turned to 90 degrees
- moved C18 30.3 mm to (150.4, 109.5), turned to -90 degrees
- moved C17 29.1 mm to (149.4, 102.5), turned to 180 degrees
- moved SW3 29.0 mm to (104.5, 139.0)
- moved C13 28.6 mm to (148.4, 99.5), turned to 90 degrees
- moved R8 28.3 mm to (104.5, 131.5)
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Routing:
- net GND: track 0.00 -> 64.7 mm
- net /MCU/BOOT: track 0.00 -> 56.6 mm
- net BAT+: track 0.00 -> 54.0 mm
- net /MCU/BAT_SENSE: track 0.00 -> 47.2 mm, vias 0 -> 3
- net /MCU/VIB_EN: track 0.00 -> 46.2 mm, vias 0 -> 2
- net /MCU/KEY: track 0.00 -> 42.0 mm
- net +3V3: track 0.00 -> 35.9 mm
- net /MCU/SWDIO: track 0.00 -> 32.4 mm, vias 0 -> 1
- net /MCU/SWCLK: track 0.00 -> 30.0 mm, vias 0 -> 1
- net /MCU/VBUS: track 0.00 -> 28.5 mm, vias 0 -> 2
- net +5V: track 0.00 -> 27.8 mm
- net /MCU/D+: track 0.00 -> 25.1 mm
- net /MCU/D-: track 0.00 -> 24.6 mm
- net /MCU/nRST: track 0.00 -> 23.6 mm
- net Net-(U5-XTO): track 0.00 -> 18.6 mm
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Other:
- board size 60 x 105 mm -> 60 x 88.5 mm

Commit message: routing complete
Parts:
- removed C14: 100p, Capacitor_SMD:C_0805_2012Metric
- removed R13, R14: 1k, Resistor_SMD:R_0805_2012Metric
- added AE3: Antenna_Loop, NetTie:NetTie-2_SMD_Pad0.5mm, F.Cu at (140.7, 99.7)
- added C37: 10p, Capacitor_SMD:C_0805_2012Metric, F.Cu at (141.4, 103.3)
- added C38: 150p, Capacitor_SMD:C_0805_2012Metric, F.Cu at (143.5, 103.3)
- added C39: 150p, Capacitor_SMD:C_0805_2012Metric, F.Cu at (133.1, 103.2)
- added R21: 0, Resistor_SMD:R_0805_2012Metric, F.Cu at (139.3, 101.3)
- added R22: 0, Resistor_SMD:R_0805_2012Metric, F.Cu at (137.3, 101.4)
- C15: value 100p -> 10p
- L3, L4: footprint Inductor_SMD:L_0402_1005Metric -> Inductor_SMD:L_0805_2012Metric_Pad1.05x1.20mm_HandSolder
- moved C33 22.6 mm to (134.7, 123.0), turned to 180 degrees
- moved J6 21.1 mm to (137.7, 123.3), turned to 0 degrees
- moved C30 20.4 mm to (134.7, 120.8), turned to 180 degrees
- moved C10 19.0 mm to (152.2, 123.7), turned to 180 degrees
- moved J5 18.1 mm to (144.5, 125.0), turned to 90 degrees
- moved C19 17.6 mm to (134.2, 106.2), turned to 180 degrees
- moved C11 17.3 mm to (147.7, 123.9), turned to 0 degrees
- moved R12 17.1 mm to (141.2, 124.2), turned to 180 degrees
- moved C13 17.0 mm to (134.2, 108.7), turned to 180 degrees
- moved Q1 16.7 mm to (154.1, 100.3)
- moved D4 16.5 mm to (154.0, 106.0)
- moved J4 16.5 mm to (158.0, 107.3)
- moved R11 16.5 mm to (154.0, 97.0)
- moved C32 14.4 mm to (147.7, 121.8), turned to 0 degrees
- moved C22 14.3 mm to (134.5, 111.5), turned to 180 degrees
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Connections:
- C15 pad 2: Net-(C15-Pad2) -> /RFID/DR2
Routing:
- net +3V3: track 35.9 -> 141.4 mm, vias 0 -> 6
- net BAT+: track 54.0 -> 139.6 mm, vias 0 -> 1
- net /MCU/NFC_SCK: track 0.00 -> 51.7 mm
- net /MCU/NFC_MOSI: track 0.00 -> 50.2 mm, vias 0 -> 2
- net /MCU/NFC_MISO: track 0.00 -> 44.2 mm, vias 0 -> 2
- net GND: track 64.7 -> 106.6 mm, vias 0 -> 55
- net /MCU/VIB_EN: track 46.2 -> 77.4 mm, vias 2 -> 4
- net /MCU/NFC_NSS: track 0.00 -> 31.0 mm, vias 0 -> 2
- net Net-(U5-RFI1): track 3.18 -> 31.9 mm
- net /MCU/NFC_IRQ: track 0.00 -> 27.2 mm, vias 0 -> 2
- net Net-(U5-RFI2): track 2.77 -> 23.5 mm
- net +5V: track 27.8 -> 46.0 mm, vias 0 -> 6
- net /MCU/PN532_NSS: track 0.00 -> 11.3 mm, vias 0 -> 1
- net /RFID/DC3: track 10.2 -> 20.1 mm, vias 0 -> 2
- net /MCU/BAT_SENSE: track 47.2 -> 56.2 mm
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- added copper zone on B.Cu, net +5V
- added copper zone on F.Cu, net +5V
- added copper zone on B.Cu, net GND
- added copper zone on F.Cu, net GND

Commit message: almost ready for fabrication
Parts:
- AE1: renamed from AE3; footprint NetTie:NetTie-2_SMD_Pad0.5mm -> Snapeda:NFC_Loop_40x30_3T
- C10: renamed from C7; value 4.3p -> 8.2p
- C11: renamed from C6; value 4.3p -> 8.2p
- U4: renamed from U1; value STM32L432KCUx -> STM32L432KBUx
- moved AE1 25.8 mm to (129.5, 76.5), turned to 0 degrees
- renumbered C35 to C1, C9 to C12, C10 to C13, C38 to C14, C39 to C15, C37 to C16, C15 to C17, C11 to C18, C12 to C19, C36 to C2, C13 to C20, C16 to C21, C17 to C22, C18 to C23, C19 to C24, C20 to C25, C21 to C26, C22 to C27, C23 to C28, C24 to C29, C34 to C3, C25 to C30, C26 to C31, C27 to C32, C28 to C33, C29 to C34, C30 to C35, C31 to C36, C32 to C37, C33 to C38, C2 to C4, C8 to C5, C1 to C6, C3 to C7, C4 to C8, C5 to C9, D3 to D1, D1 to D3, J7 to J3, J3 to J5, J5 to J6, J6 to J7, L3 to L1, L4 to L2, R19 to R10, R20 to R11, R7 to R12, R8 to R13, R9 to R14, R10 to R15, R11 to R16, R12 to R17, R15 to R18, R21 to R19, R22 to R20, R16 to R7, R17 to R8, R18 to R9, U6 to U1, Y2 to Y1, Y1 to Y2
Routing:
- net Net-(AE1-Pad1): track 0.00 -> 7.06 mm
- net Net-(AE1-Pad2): track 0.00 -> 5.84 mm

Commit message: Mounting holes and WX logo added
Parts:
- added G***: LOGO, External:wx, F.Cu at (104.8, 99.5)
- added REF**: Mounting_Wuerth_WA-SMSR-3.2mm_H10.6mm_ReverseMount_97751069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, Mounting_Wuerth:Mounting_Wuerth_WA-SMSR-3.2mm_H10.6mm_ReverseMount_9775106960, F.Cu at (104.2, 60.8)
- added REF**: Mounting_Wuerth_WA-SMSR-3.2mm_H10.6mm_ReverseMount_97751069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, Mounting_Wuerth:Mounting_Wuerth_WA-SMSR-3.2mm_H10.6mm_ReverseMount_9775106960, F.Cu at (104.2, 106.8)
- added REF**: Mounting_Wuerth_WA-SMSR-3.2mm_H10.6mm_ReverseMount_97751069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, Mounting_Wuerth:Mounting_Wuerth_WA-SMSR-3.2mm_H10.6mm_ReverseMount_9775106960, F.Cu at (155.8, 140.8)
- added REF**: Mounting_Wuerth_WA-SMSR-3.2mm_H10.6mm_ReverseMount_97751069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, Mounting_Wuerth:Mounting_Wuerth_WA-SMSR-3.2mm_H10.6mm_ReverseMount_9775106960, F.Cu at (155.8, 60.8)
- moved TH1 7.37 mm to (148.1, 142.3)
Routing:
- net Net-(U2-THERM): track 3.82 -> 8.74 mm
- net unconnected-(U4-PA1-Pad7): track 0.00 -> 4.08 mm, vias 0 -> 1
- net unconnected-(U4-PA8-Pad18): track 0.00 -> 3.41 mm
- net unconnected-(U4-PA6-Pad12): track 0.00 -> 3.00 mm
- net unconnected-(U4-PA5-Pad11): track 0.00 -> 2.97 mm, vias 0 -> 1
- net unconnected-(U4-PA10-Pad20): track 0.00 -> 2.10 mm
- net /MCU/VIB_EN: track 77.4 -> 78.5 mm
Other:
- board text added: "BOOT"
- board text added: "PWR"
- board text added: "RST"
