File: PCB/Attendance Management System.kicad_pcb (KiCad board)
At the start: 2 copper layers, 60 x 88.5 mm, 93 parts, among them J1 USB-C, J2 BATTERY, J3 PN532, J4 VIB_MOTOR, J5 SWD, J6 CSO, J7 CSI, Q1 AO3400A, SW1 RST, SW2 BOOT0, SW3 POWER, U1 USBLC6-2SC6, U2 MCP73833-xxx-UN, U3 TPS7A0233PDBVR, U4 STM32L432KBUx, U5 ST25R3916-AQWT, Y1 32.768k, Y2 27.12MHz

Commit message: Move the through-hole parts to the back of the board
J2, J5, TH1 and the J3/J4 footprints go on B.Cu so the front stays flat for the slim enclosure.
Parts:
- J2, J3, J4, J5, TH1: moved to B.Cu
- turned J3 to 90 degrees
- turned J4 to 0 degrees
- turned J5 to 0 degrees
