File: PCB/_restore_backup_2026-09-25T09-19-25-262/mcu.kicad_sch (KiCad schematic)
At the start: 27 parts, among them J3 SW, J4 MOT, Q1 AO3400A, SW1 RST, SW2 BOOT, SW3 KEY, U1 STM32L432KCUx, Y2 32kHz

Commit message: Schematic is almost ready
Other:
- moved on the sheet: R18, R19
Changed lines of the file:
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@@
 	)
 	(junction
-		(at 45.72 44.45)
+		(at 44.45 44.45)
 		(diameter 0)
 		(color 0 0 0 0)
@@
 	(wire
 		(pts
-			(xy 45.72 30.48) (xy 45.72 34.29)
+			(xy 44.45 30.48) (xy 44.45 34.29)
 		)
 		(stroke
@@
 	(wire
 		(pts
-			(xy 45.72 44.45) (xy 45.72 46.99)
+			(xy 44.45 44.45) (xy 44.45 46.99)
 		)
 		(stroke
@@
 	(wire
 		(pts
-			(xy 45.72 41.91) (xy 45.72 44.45)
+			(xy 44.45 41.91) (xy 44.45 44.45)
 		)
 		(stroke
@@
 	(wire
 		(pts
-			(xy 45.72 44.45) (xy 53.34 44.45)
+			(xy 44.45 44.45) (xy 52.07 44.45)
 		)
 		(stroke
@@
 	(wire
 		(pts
-			(xy 45.72 54.61) (xy 45.72 59.69)
+			(xy 44.45 54.61) (xy 44.45 59.69)
 		)
 		(stroke
@@
 	)
 	(label "VBUS"
-		(at 53.34 44.45 0)
+		(at 52.07 44.45 0)
 		(effects
 			(font
@@
 	(symbol
 		(lib_id "Device:R")
-		(at 45.72 38.1 0)
+		(at 44.45 38.1 0)
 		(unit 1)
 		(body_style 1)
@@
 		(dnp no)
 		(property "Reference" "R18"
-			(at 48.768 36.83 0)
+			(at 47.498 36.83 0)
 			(show_name no)
 			(do_not_autoplace no)
@@
 		)
 		(property "Value" "4M7"
-			(at 49.022 38.862 0)
+			(at 47.752 38.862 0)
 			(show_name no)
 			(do_not_autoplace no)
@@
 		)
 		(property "Footprint" "Resistor_SMD:R_0805_2012Metric"
-			(at 43.942 38.1 90)
+			(at 42.672 38.1 90)
 			(hide yes)
 			(show_name no)
@@
 		)
 		(property "Datasheet" ""
-			(at 45.72 38.1 0)
+			(at 44.45 38.1 0)
 			(hide yes)
 			(show_name no)
@@
 		)
 		(property "Description" "Resistor"
-			(at 45.72 38.1 0)
+			(at 44.45 38.1 0)
 			(hide yes)
 			(show_name no)
@@
 	(symbol
 		(lib_id "power:+3V3")
-		(at 45.72 30.48 0)
+		(at 44.45 30.48 0)
 		(unit 1)
 		(body_style 1)
@@
 		(dnp no)
 		(property "Reference" "#PWR065"
-			(at 45.72 34.29 0)
+			(at 44.45 34.29 0)
 			(hide yes)
 			(show_name no)
@@
 		)
 		(property "Value" "+5V"
-			(at 45.72 24.892 90)
+			(at 44.45 24.892 90)
 			(show_name no)
 			(do_not_autoplace no)
@@
 		)
 		(property "Footprint" ""
-			(at 45.72 30.48 0)
+			(at 44.45 30.48 0)
 			(hide yes)
 			(show_name no)
@@
 		)
 		(property "Datasheet" ""
-			(at 45.72 30.48 0)
+			(at 44.45 30.48 0)
 			(hide yes)
 			(show_name no)
@@
 		)
 		(property "Description" "Power symbol creates a global label with name \"+3V3\""
-			(at 45.72 30.48 0)
+			(at 44.45 30.48 0)
 			(hide yes)
 			(show_name no)
@@
 	(symbol
 		(lib_id "Device:R")
-		(at 45.72 50.8 0)
+		(at 44.45 50.8 0)
 		(unit 1)
 		(body_style 1)
@@
 		(dnp no)
 		(property "Reference" "R19"
-			(at 48.768 49.53 0)
+			(at 47.498 49.53 0)
 			(show_name no)
 			(do_not_autoplace no)
@@
 		)
 		(property "Value" "4M7"
-			(at 48.768 51.562 0)
+			(at 47.498 51.562 0)
 			(show_name no)
 			(do_not_autoplace no)
@@
 		)
 		(property "Footprint" "Resistor_SMD:R_0805_2012Metric"
-			(at 43.942 50.8 90)
+			(at 42.672 50.8 90)
 			(hide yes)
 			(show_name no)
@@
 		)
 		(property "Datasheet" ""
-			(at 45.72 50.8 0)
+			(at 44.45 50.8 0)
 			(hide yes)
 			(show_name no)
@@
 		)
 		(property "Description" "Resistor"
-			(at 45.72 50.8 0)
+			(at 44.45 50.8 0)
 			(hide yes)
 			(show_name no)
@@
 	(symbol
 		(lib_id "power:GND")
-		(at 45.72 59.69 0)
+		(at 44.45 59.69 0)
 		(unit 1)
 		(body_style 1)
@@
 		(fields_autoplaced yes)
 		(property "Reference" "#PWR066"
-			(at 45.72 66.04 0)
+			(at 44.45 66.04 0)
 			(hide yes)
 			(show_name no)
@@
 		)
 		(property "Value" "GND"
-			(at 45.72 64.77 0)
+			(at 44.45 64.77 0)
 			(show_name no)
 			(do_not_autoplace no)
@@
 		)
 		(property "Footprint" ""
-			(at 45.72 59.69 0)
+			(at 44.45 59.69 0)
 			(hide yes)
 			(show_name no)
@@
 		)
 		(property "Datasheet" ""
-			(at 45.72 59.69 0)
+			(at 44.45 59.69 0)
 			(hide yes)
 			(show_name no)
@@
 		)
 		(property "Description" "Power symbol creates a global label with name \"GND\" , ground"
-			(at 45.72 59.69 0)
+			(at 44.45 59.69 0)
 			(hide yes)
 			(show_name no)
